Commit message: modified urdf

File: urdf/rosbot.xacro (robot description, xacro)
@@ -278,5 +278,5 @@
       <origin xyz="${scale_bot*0.01} 0 ${scale_bot*0.004}" rpy="1.5707 0 1.5707"/>
       <geometry>
-        <mesh filename="package://EXPROBLAB_Assignment2/meshes/astra.stl" scale="${scale_bot*0.001} ${scale_bot*0.001} ${scale_bot*0.001}" />
+        <mesh filename="package://EXPROBLAB_Assignment2/meshes/astra.stl" scale="${scale_bot*0.001/2} ${scale_bot*0.001/2} ${scale_bot*0.001/2}" />
       </geometry>
       <material name="Black"/>

File: urdf/youbot_arm/arm.urdf.xacro (robot description, xacro)
@@ -179,5 +179,5 @@
       <parent link="${name}_link_4"/>
       <child link="${name}_link_5"/>
-      <axis xyz="0 0 -1" />
+      <axis xyz="0 0 1" />
       <!--<calibration rising="${arm_5_ref}" falling="${arm_5_ref}"/>-->
       <dynamics damping="1" friction="1" />

File: urdf/youbot_arm/limits.urdf.xacro (robot description, xacro)
@@ -8,5 +8,5 @@
   <!-- up limits [rad] -->
   <xacro:property name="joint_1_limit_up" value="${M_PI}" />
-  <xacro:property name="joint_2_limit_up" value="2" />
+  <xacro:property name="joint_2_limit_up" value="${M_PI}" />
   <xacro:property name="joint_3_limit_up" value="0" />
   <xacro:property name="joint_4_limit_up" value="2.5" />
@@ -20,5 +20,5 @@
   <!-- up limits soft [rad] -->
   <xacro:property name="joint_1_limit_up_soft" value="${M_PI - threshold}" />
-  <xacro:property name="joint_2_limit_up_soft" value="${2 - threshold}" />
+  <xacro:property name="joint_2_limit_up_soft" value="${M_PI - threshold}" />
   <xacro:property name="joint_3_limit_up_soft" value="${0 - threshold}" />
   <xacro:property name="joint_4_limit_up_soft" value="${2.5 - threshold}" />
@@ -31,10 +31,10 @@
   <xacro:property name="joint_5_limit_down_soft" value="${-M_PI + threshold}" />
   <!-- dynamic properties : mass (kg) Alu data sheet -->
-  <xacro:property name="link_0_mass" value="${scale*0.845}" />
-  <xacro:property name="link_1_mass" value="${scale*2.412}" />
-  <xacro:property name="link_2_mass" value="${scale*1.155}" />
-  <xacro:property name="link_3_mass" value="${scale*0.934}" />
-  <xacro:property name="link_4_mass" value="${scale*0.877}" />
-  <xacro:property name="link_5_mass" value="${scale*0.251}" />
+  <xacro:property name="link_0_mass" value="${0.845}" />
+  <xacro:property name="link_1_mass" value="${2.412}" />
+  <xacro:property name="link_2_mass" value="${1.155}" />
+  <xacro:property name="link_3_mass" value="${0.934}" />
+  <xacro:property name="link_4_mass" value="${0.877}" />
+  <xacro:property name="link_5_mass" value="${0.251}" />
   <!--<xacro:property name="link_0_mass" value="0.845" />
   <xacro:property name="link_1_mass" value="0.1" />

Commit message: robot modifications

File: urdf/rosbot.xacro (robot description, xacro)
@@ -3,5 +3,5 @@
   xmlns:xacro="http://www.ros.org/wiki/xacro">
   <xacro:arg name="robot_namespace" default="rosbot"/>
-  <xacro:property name="scale_bot" value="3"/>
+  <xacro:property name="scale_bot" value="3.0"/>
   <xacro:include filename="$(find EXPROBLAB_Assignment2)/urdf/materials.xacro" />
   <xacro:include filename="$(find EXPROBLAB_Assignment2)/urdf/rosbot.gazebo" />
@@ -302,19 +302,16 @@
   <link name="camera_depth_frame">
   </link>
-<!--
   <joint name="rplidar_joint" type="fixed">
     <axis xyz="0 1 0" />
-    <origin xyz="0.02 0 0.058" rpy="0 0 3.14"/>
+    <origin xyz="${scale_bot*0.1} 0 ${scale_bot*0.058/4}" rpy="0 0 3.14"/>
     <parent link="body_link"/>
     <child link="laser"/>
   </joint>
--->
   <!-- rplidar Laser -->
-  <!--
   <link name="laser">
     <collision>
       <origin xyz="0 0 0" rpy="1.5707 0 4.71"/>
       <geometry>
-        <mesh filename="package://EXPROBLAB_Assignment2/meshes/rplidar.stl" scale="0.001 0.001 0.001" />
+        <mesh filename="package://EXPROBLAB_Assignment2/meshes/rplidar.stl" scale="${scale_bot*0.001} ${scale_bot*0.001} ${scale_bot*0.001}" />
       </geometry>
     </collision>
@@ -322,10 +319,10 @@
       <origin xyz="0 0 0" rpy="1.5707 0 4.71"/>
       <geometry>
-        <mesh filename="package://EXPROBLAB_Assignment2/meshes/rplidar.stl" scale="0.001 0.001 0.001" />
-      </geometry>
-      <material name="Black"/>
-    </visual>
-    <inertial>
-      <mass value="1e-5" />
+        <mesh filename="package://EXPROBLAB_Assignment2/meshes/rplidar.stl" scale="${scale_bot*0.001} ${scale_bot*0.001} ${scale_bot*0.001}" />
+      </geometry>
+      <material name="Black"/>
+    </visual>
+    <inertial>
+      <mass value="${scale_bot*1e-5}" />
       <origin xyz="0 0 0" rpy="1.5707 0 4.71"/>
       <inertia ixx="0" ixy="0" ixz="0" iyy="0" iyz="0" izz="0" />
@@ -334,5 +331,5 @@
   <joint name="range_fl_joint" type="fixed">
     <axis xyz="0 1 0" />
-    <origin xyz="0.1 0.05 0.01" rpy="0 0 0.13 "/>
+    <origin xyz="${scale_bot*0.1} ${scale_bot*0.05} ${scale_bot*0.01}" rpy="0 0 0.13 "/>
     <parent link="body_link"/>
     <child link="range_fl"/>
@@ -341,5 +338,5 @@
   <joint name="range_fr_joint" type="fixed">
     <axis xyz="0 1 0" />
-    <origin xyz="0.1 -0.05 0.01" rpy="0 0 -0.13 "/>
+    <origin xyz="${scale_bot*0.1} ${scale_bot*-0.05} ${scale_bot*0.01}" rpy="0 0 -0.13 "/>
     <parent link="body_link"/>
     <child link="range_fr"/>
@@ -348,5 +345,5 @@
   <joint name="range_rl_joint" type="fixed">
     <axis xyz="0 1 0" />
-    <origin xyz="-0.1 0.05 0.01" rpy="0 0 3.01 "/>
+    <origin xyz="${scale_bot*-0.1} ${scale_bot*0.05} ${scale_bot*0.01}" rpy="0 0 3.01 "/>
     <parent link="body_link"/>
     <child link="range_rl"/>
@@ -355,9 +352,8 @@
   <joint name="range_rr_joint" type="fixed">
     <axis xyz="0 1 0" />
-    <origin xyz="-0.1 -0.05 0.01" rpy="0 0 3.27 "/>
+    <origin xyz="${scale_bot*-0.1} ${scale_bot*-0.05} ${scale_bot*0.01}" rpy="0 0 3.27 "/>
     <parent link="body_link"/>
     <child link="range_rr"/>
   </joint>
   <link name="range_rr"></link>
--->
 </robot>

File: urdf/youbot_arm/arm.urdf.xacro (robot description, xacro)
@@ -7,5 +7,5 @@
   <xacro:include filename="$(find EXPROBLAB_Assignment2)/urdf/youbot_arm/arm.transmission.xacro" />
   <xacro:include filename="$(find EXPROBLAB_Assignment2)/urdf/youbot_arm/limits.urdf.xacro" />
-  <xacro:property name="scale_robot" value="3"/>
+  <xacro:property name="scale_robot" value="3.0"/>
   <xacro:property name="scale" value="${scale_robot*0.6}"/>
   <!-- specifies the offset to include the 10mm table flange and the 3.225cm model offset -->

File: urdf/youbot_arm/limits.urdf.xacro (robot description, xacro)
@@ -3,5 +3,5 @@
   <!-- common properties -->
   <xacro:property name="M_PI" value="3.1415926535897931" />
-  <xacro:property name="scale_robot" value="3"/>
+  <xacro:property name="scale_robot" value="3.0"/>
   <xacro:property name="scale" value="${scale_robot*0.6}"/>
   <xacro:property name="threshold" value="${0}" />

Commit message: added kp kd

File: urdf/rosbot.xacro (robot description, xacro)
@@ -16,10 +16,10 @@
     <pose>0 0 ${scale_bot*0.1} 0 0 0</pose>
     <inertial>
-      <mass value="${scale_bot*5}"/>
+      <mass value="5"/>
       <origin xyz="0 0 ${scale_bot*0.04}" rpy=" 0 0 0"/>
       <inertia
-      ixx="${scale_bot*0.01}" ixy="${scale_bot*0.01}" ixz="0"
-      iyy="${scale_bot*0.01}" iyz="${scale_bot*0.01}"
-      izz="${scale_bot*0.01}"
+      ixx="0.01" ixy="0.01" ixz="0"
+      iyy="0.01" iyz="0.01"
+      izz="0.01"
       />
     </inertial>
@@ -47,5 +47,5 @@
     <pose>0 0 0 0 0 0</pose>
     <inertial>
-      <mass value="${scale_bot*0.01}"/>
+      <mass value="0.01"/>
       <origin xyz="0 0 ${scale_bot*0.055}" rpy=" 0 0 0"/>
       <inertia
@@ -67,5 +67,5 @@
   <link name="front_left_wheel">
     <collision>
-      <origin xyz="0 ${scale_bot*-0.014} 0" rpy="${pi/2} 0 0"/>
+      <origin xyz="0 0 0" rpy="${pi/2} 0 0"/>
       <geometry>
         <cylinder length="${scale_bot*0.036}" radius="${scale_bot*0.04}"/>
@@ -76,4 +76,6 @@
             <mu>10</mu>
             <mu2>10</mu2>
+            <kp value="10000000.0" />
+            <kd value="0.0" />
           </ode>
         </friction>
@@ -89,9 +91,9 @@
     <inertial>
       <origin xyz="0 0 0" rpy="0 1.5707 1.5707"/>
-      <mass value="${scale_bot*0.5}"/>
-      <inertia
-      ixx="${scale_bot*0.001}" ixy="0.0" ixz="0"
-      iyy="${scale_bot*0.001}" iyz="0.0"
-      izz="${scale_bot*0.001}"
+      <mass value="0.5"/>
+      <inertia
+      ixx="0.001" ixy="0.0" ixz="0"
+      iyy="0.001" iyz="0.0"
+      izz="0.001"
       />
     </inertial>
@@ -99,5 +101,5 @@
   <link name="front_right_wheel">
     <collision>
-      <origin xyz="0 ${scale_bot*0.014} 0" rpy="${pi/2} 0 0"/>
+      <origin xyz="0 0 0" rpy="0 0 -1.5707"/>
       <geometry>
         <cylinder length="${scale_bot*0.036}" radius="${scale_bot*0.04}"/>
@@ -108,4 +110,6 @@
             <mu>10</mu>
             <mu2>10</mu2>
+            <kp value="10000000.0" />
+            <kd value="0.0" />
           </ode>
         </friction>
@@ -121,9 +125,9 @@
     <inertial>
       <origin xyz="0 0 0" rpy="0 1.5707 1.5707"/>
-      <mass value="${scale_bot*0.5}"/>
-      <inertia
-      ixx="${scale_bot*0.001}" ixy="0.0" ixz="0"
-      iyy="${scale_bot*0.001}" iyz="0.0"
-      izz="${scale_bot*0.001}"
+      <mass value="0.5"/>
+      <inertia
+      ixx="0.001" ixy="0.0" ixz="0"
+      iyy="0.001" iyz="0.0"
+      izz="0.001"
       />
     </inertial>
@@ -131,5 +135,5 @@
   <link name="rear_left_wheel">
     <collision>
-      <origin xyz="0 ${scale_bot*-0.014} 0" rpy="${pi/2} 0 0"/>
+      <origin xyz="0 0 0" rpy="0 0 1.5707"/>
       <geometry>
         <cylinder length="${scale_bot*0.036}" radius="${scale_bot*0.04}"/>
@@ -140,4 +144,6 @@
             <mu>10</mu>
             <mu2>10</mu2>
+            <kp value="10000000.0" />
+            <kd value="0.0" />
           </ode>
         </friction>
@@ -153,9 +159,9 @@
     <inertial>
       <origin xyz="0 0 0" rpy="0 1.5707 1.5707"/>
-      <mass value="${scale_bot*0.5}"/>
-      <inertia
-      ixx="${scale_bot*0.001}" ixy="0.0" ixz="0"
-      iyy="${scale_bot*0.001}" iyz="0.0"
-      izz="${scale_bot*0.001}"
+      <mass value="0.5"/>
+      <inertia
+      ixx="0.001" ixy="0.0" ixz="0"
+      iyy="0.001" iyz="0.0"
+      izz="0.001"
       />
     </inertial>
@@ -163,5 +169,5 @@
   <link name="rear_right_wheel">
     <collision>
-      <origin xyz="0 ${scale_bot*0.014} 0" rpy="${pi/2} 0 0"/>
+      <origin xyz="0 0 0" rpy="0 0 -1.5707"/>
       <geometry>
         <cylinder length="${scale_bot*0.036}" radius="${scale_bot*0.04}"/>
@@ -172,4 +178,6 @@
             <mu>10</mu>
             <mu2>10</mu2>
+            <kp value="10000000.0" />
+            <kd value="0.0" />
           </ode>
         </friction>
@@ -185,9 +193,9 @@
     <inertial>
       <origin xyz="0 0 0" rpy="0 1.5707 1.5707"/>
-      <mass value="${scale_bot*0.5}"/>
-      <inertia
-      ixx="${scale_bot*0.001}" ixy="0.0" ixz="0"
-      iyy="${scale_bot*0.001}" iyz="0.0"
-      izz="${scale_bot*0.001}"
+      <mass value="0.5"/>
+      <inertia
+      ixx="0.001" ixy="0.0" ixz="0"
+      iyy="0.001" iyz="0.0"
+      izz="0.001"
       />
     </inertial>
@@ -283,5 +291,5 @@
     </visual>
     <inertial>
-      <mass value="${scale_bot*1e-5}" />
+      <mass value="1e-5" />
       <origin xyz="0 0 0" rpy="0 0 0"/>
       <inertia ixx="0" ixy="0" ixz="0" iyy="0" iyz="0" izz="0" />
@@ -324,5 +332,5 @@
     </visual>
     <inertial>
-      <mass value="${scale_bot*1e-5}" />
+      <mass value="1e-5" />
       <origin xyz="0 0 0" rpy="1.5707 0 4.71"/>
       <inertia ixx="0" ixy="0" ixz="0" iyy="0" iyz="0" izz="0" />

File: urdf/youbot_arm/arm.transmission.xacro (robot description, xacro)
@@ -6,5 +6,5 @@
   <!-- reduction ratio doesn't affect the model-->
   <!-- reduction ratio must not to be 0-->
-  <xacro:property name="scale" value="0.6"/>
+  <xacro:property name="scale" value="0.5"/>
   <xacro:macro name="youbot_arm_transmission" params="name">
     <transmission name="${name}_trans_1">

File: urdf/youbot_arm/arm.urdf.xacro (robot description, xacro)
@@ -8,5 +8,5 @@
   <xacro:include filename="$(find EXPROBLAB_Assignment2)/urdf/youbot_arm/limits.urdf.xacro" />
   <xacro:property name="scale_robot" value="3.0"/>
-  <xacro:property name="scale" value="${scale_robot*0.6}"/>
+  <xacro:property name="scale" value="${scale_robot*0.5}"/>
   <!-- specifies the offset to include the 10mm table flange and the 3.225cm model offset -->
   <xacro:macro name="youbot_arm" params="parent name">
@@ -22,5 +22,5 @@
         <!--<origin xyz="0 0 0" rpy="0 0 0"/>-->
         <mass value="${link_0_mass}"/>
-        <inertia ixx="${scale*0.01}" ixy="0" ixz="0" iyy="${scale*0.01}" iyz="0" izz="${scale*0.01}" />
+        <inertia ixx="0.01" ixy="0" ixz="0" iyy="0.01" iyz="0" izz="0.01" />
       </inertial>
       <visual>

File: urdf/youbot_arm/limits.urdf.xacro (robot description, xacro)
@@ -4,5 +4,5 @@
   <xacro:property name="M_PI" value="3.1415926535897931" />
   <xacro:property name="scale_robot" value="3.0"/>
-  <xacro:property name="scale" value="${scale_robot*0.6}"/>
+  <xacro:property name="scale" value="${scale_robot*0.5}"/>
   <xacro:property name="threshold" value="${0}" />
   <!-- up limits [rad] -->
@@ -49,25 +49,25 @@
   <xacro:macro name="link_default_inertia_tensor">
     <origin xyz="0 0 0" rpy="0 0 0" />
-    <inertia ixx="${scale*0.1}" ixy="0" ixz="0" iyy="${scale*0.1}" iyz="0" izz="${scale*0.1}" />
+    <inertia ixx="0.1" ixy="0" ixz="0" iyy="0.1" iyz="0" izz="0.1" />
   </xacro:macro>
   <xacro:macro name="link_1_inertia_tensor">
     <origin xyz="${scale*14.89/1000} ${scale*2.13/1000} ${scale*2.13/1000}" rpy="0 0 0" />
-    <inertia ixx="${scale*0.003863}" ixy="${scale*-0.000979}" ixz="0.000000" iyy="${scale*0.006196}" iyz="0.000000" izz="${scale*0.006369}" />
+    <inertia ixx="0.003863" ixy="-0.000979" ixz="0.000000" iyy="0.006196" iyz="0.000000" izz="0.006369" />
   </xacro:macro>
   <xacro:macro name="link_2_inertia_tensor">
     <origin xyz="${scale*104.53/1000} ${scale*1.7/1000} ${scale*-2.97/1000}" rpy="0 0 0" />
-    <inertia ixx="${scale*0.000823}" ixy="0.000000" ixz="-0.000000" iyy="${scale*0.004447}" iyz ="0.000000" izz="${scale*0.004439}" />
+    <inertia ixx="0.000823" ixy="0.000000" ixz="-0.000000" iyy="0.004447" iyz ="0.000000" izz="0.004439" />
   </xacro:macro>
   <xacro:macro name="link_3_inertia_tensor">
     <origin xyz="${scale*0.1/1000} ${scale*96.7/1000} ${scale*21.07/1000}" rpy="0 0 0" />
-    <inertia ixx="${scale*0.002459}" ixy="0.000000" ixz="0.000000" iyy="${scale*0.002571}" iyz="-0.000000" izz="${scale*0.000535}" />
+    <inertia ixx="0.002459" ixy="0.000000" ixz="0.000000" iyy="0.002571" iyz="-0.000000" izz="0.000535" />
   </xacro:macro>
   <xacro:macro name="link_4_inertia_tensor">
     <origin xyz="${scale*0.11/1000} ${scale*51.03/1000} ${scale*-23.19/1000}" rpy="0 0 0"  />
-    <inertia ixx="${scale*0.000869}" ixy="0.000000" ixz="-0.000000" iyy="${scale*0.001173}" iyz="${scale*-0.000231}" izz="${scale*0.001091}" />
+    <inertia ixx="0.000869" ixy="0.000000" ixz="-0.000000" iyy="0.001173" iyz="-0.000231" izz="0.001091" />
   </xacro:macro>
   <xacro:macro name="link_5_inertia_tensor">
     <origin xyz="${scale*0/1000} ${scale*1.15/1000} ${scale*-16.83/1000}" rpy="0 0 0" />
-    <inertia ixx="${scale*0.000280}" ixy="0.000000" ixz="0.000000" iyy="${scale*0.000339}" iyz="0.000000" izz="${scale*0.000119}" />
+    <inertia ixx="0.000280" ixy="0.000000" ixz="0.000000" iyy="0.000339" iyz="0.000000" izz="0.000119" />
   </xacro:macro>
 </robot>

Commit message: adjustment

File: urdf/rosbot.xacro (robot description, xacro)
@@ -67,5 +67,5 @@
   <link name="front_left_wheel">
     <collision>
-      <origin xyz="0 0 0" rpy="${pi/2} 0 0"/>
+      <origin xyz="0 ${scale_bot*-0.014} 0" rpy="${pi/2} 0 0"/>
       <geometry>
         <cylinder length="${scale_bot*0.036}" radius="${scale_bot*0.04}"/>
@@ -90,5 +90,5 @@
     </visual>
     <inertial>
-      <origin xyz="0 0 0" rpy="0 1.5707 1.5707"/>
+      <origin xyz="0 0 0" rpy="${pi/2} 0 0"/>
       <mass value="0.5"/>
       <inertia
@@ -101,5 +101,5 @@
   <link name="front_right_wheel">
     <collision>
-      <origin xyz="0 0 0" rpy="0 0 -1.5707"/>
+      <origin xyz="0 ${scale_bot*0.014} 0" rpy="${pi/2} 0 0"/>
       <geometry>
         <cylinder length="${scale_bot*0.036}" radius="${scale_bot*0.04}"/>
@@ -135,5 +135,5 @@
   <link name="rear_left_wheel">
     <collision>
-      <origin xyz="0 0 0" rpy="0 0 1.5707"/>
+      <origin xyz="0 ${scale_bot*-0.014} 0" rpy="${pi/2} 0 0"/>
       <geometry>
         <cylinder length="${scale_bot*0.036}" radius="${scale_bot*0.04}"/>
@@ -169,5 +169,5 @@
   <link name="rear_right_wheel">
     <collision>
-      <origin xyz="0 0 0" rpy="0 0 -1.5707"/>
+      <origin xyz="0 ${scale_bot*0.014} 0" rpy="${pi/2} 0 0"/>
       <geometry>
         <cylinder length="${scale_bot*0.036}" radius="${scale_bot*0.04}"/>
@@ -312,5 +312,5 @@
   <joint name="rplidar_joint" type="fixed">
     <axis xyz="0 1 0" />
-    <origin xyz="${scale_bot*0.1} 0 ${scale_bot*0.058/4}" rpy="0 0 3.14"/>
+    <origin xyz="${scale_bot*0.1} 0 ${scale_bot*0.0584}" rpy="0 0 3.14"/>
     <parent link="body_link"/>
     <child link="laser"/>
@@ -339,5 +339,5 @@
   <joint name="range_fl_joint" type="fixed">
     <axis xyz="0 1 0" />
-    <origin xyz="${scale_bot*0.1} ${scale_bot*0.05} ${scale_bot*0.01}" rpy="0 0 0.13 "/>
+    <origin xyz="${scale_bot*0.1} ${scale_bot*0.05} ${scale_bot*0.05}" rpy="0 0 0.13 "/>
     <parent link="body_link"/>
     <child link="range_fl"/>
