Commit message: modifed urdf and launch

File: urdf/rosbot.xacro (robot description, xacro)
@@ -3,16 +3,10 @@
   xmlns:xacro="http://www.ros.org/wiki/xacro">
   <xacro:arg name="robot_namespace" default="rosbot"/>
-  <xacro:property name="scale_bot" value="3.0"/>
+  <xacro:property name="scale_bot" value="1.0"/>
   <xacro:include filename="$(find EXPROBLAB_Assignment2)/urdf/materials.xacro" />
   <xacro:include filename="$(find EXPROBLAB_Assignment2)/urdf/rosbot.gazebo" />
   <xacro:include filename="$(find EXPROBLAB_Assignment2)/urdf/youbot_arm/arm.urdf.xacro" />
-  <link name="base_link"></link>
-  <joint name="base_link_joint" type="fixed">
-    <origin xyz="0 0 0" rpy="0 0 0"/>
-    <parent link="base_link"/>
-    <child link="body_link"/>
-  </joint>
-  <link name='body_link'>
-    <pose>0 0 ${scale_bot*0.1} 0 0 0</pose>
+  <link name='base_link'>
+    <pose>0 0 0.1 0 0 0</pose>
     <inertial>
       <mass value="5"/>
@@ -24,5 +18,5 @@
       />
     </inertial>
-    <collision>
+    <collision name='collision'>
       <origin xyz="0 0 ${scale_bot*0.02}" rpy="0 0 0"/>
       <geometry>
@@ -30,10 +24,9 @@
       </geometry>
     </collision>
-    <visual>
+    <visual name='base_link_visual'>
       <origin xyz="0 0 ${scale_bot*-0.02}" rpy=" 1.5707 0 1.5707"/>
       <geometry>
         <mesh filename="package://EXPROBLAB_Assignment2/meshes/box.stl" scale="${scale_bot*0.001} ${scale_bot*0.001} ${scale_bot*0.001}" />
       </geometry>
-      <material name="White"/>
     </visual>
   </link>
@@ -41,5 +34,5 @@
     <axis xyz="0 1 0" />
     <origin xyz="0 0 0" rpy="0 0 0"/>
-    <parent link="body_link"/>
+    <parent link="base_link"/>
     <child link="top"/>
   </joint>
@@ -67,7 +60,7 @@
   <link name="front_left_wheel">
     <collision>
-      <origin xyz="0 ${scale_bot*-0.014} 0" rpy="${pi/2} 0 0"/>
-      <geometry>
-        <cylinder length="${scale_bot*0.036}" radius="${scale_bot*0.04}"/>
+      <origin xyz="0 0 0" rpy="0 0 1.5707"/>
+      <geometry>
+        <mesh filename="package://EXPROBLAB_Assignment2/meshes/wheel.stl" scale="${scale_bot*0.001} ${scale_bot*0.001} ${scale_bot*0.001}" />
       </geometry>
       <surface>
@@ -90,5 +83,5 @@
     </visual>
     <inertial>
-      <origin xyz="0 0 0" rpy="${pi/2} 0 0"/>
+      <origin xyz="0 0 0" rpy="0 1.5707 1.5707"/>
       <mass value="0.5"/>
       <inertia
@@ -101,7 +94,7 @@
   <link name="front_right_wheel">
     <collision>
-      <origin xyz="0 ${scale_bot*0.014} 0" rpy="${pi/2} 0 0"/>
-      <geometry>
-        <cylinder length="${scale_bot*0.036}" radius="${scale_bot*0.04}"/>
+      <origin xyz="0 0 0" rpy="0 0 -1.5707"/>
+      <geometry>
+        <mesh filename="package://EXPROBLAB_Assignment2/meshes/wheel.stl" scale="${scale_bot*0.001} ${scale_bot*0.001} ${scale_bot*0.001}" />
       </geometry>
       <surface>
@@ -135,7 +128,7 @@
   <link name="rear_left_wheel">
     <collision>
-      <origin xyz="0 ${scale_bot*-0.014} 0" rpy="${pi/2} 0 0"/>
-      <geometry>
-        <cylinder length="${scale_bot*0.036}" radius="${scale_bot*0.04}"/>
+      <origin xyz="0 0 0" rpy="0 0 1.5707"/>
+      <geometry>
+        <mesh filename="package://EXPROBLAB_Assignment2/meshes/wheel.stl" scale="${scale_bot*0.001} ${scale_bot*0.001} ${scale_bot*0.001}" />
       </geometry>
       <surface>
@@ -169,7 +162,7 @@
   <link name="rear_right_wheel">
     <collision>
-      <origin xyz="0 ${scale_bot*0.014} 0" rpy="${pi/2} 0 0"/>
-      <geometry>
-        <cylinder length="${scale_bot*0.036}" radius="${scale_bot*0.04}"/>
+      <origin xyz="0 0 0" rpy="0 0 -1.5707"/>
+      <geometry>
+        <mesh filename="package://EXPROBLAB_Assignment2/meshes/wheel.stl" scale="${scale_bot*0.001} ${scale_bot*0.001} ${scale_bot*0.001}" />
       </geometry>
       <surface>
@@ -204,5 +197,5 @@
     <origin xyz="${scale_bot*0.05} ${scale_bot*0.11} 0" rpy="0 0 0"/>
     <child link="front_left_wheel"/>
-    <parent link="body_link"/>
+    <parent link="base_link"/>
     <axis xyz="0 1 0" rpy="0 0 0"/>
     <limit effort="1" velocity="10"/>
@@ -221,5 +214,5 @@
     <origin xyz="${scale_bot*0.05} ${scale_bot*-0.11} 0" rpy="0 0 0"/>
     <child link="front_right_wheel"/>
-    <parent link="body_link"/>
+    <parent link="base_link"/>
     <axis xyz="0 1 0" rpy="0 0 0"/>
     <limit effort="1" velocity="10"/>
@@ -238,5 +231,5 @@
     <origin xyz="${scale_bot*-0.055} ${scale_bot*0.11} 0" rpy="0 0 0"/>
     <child link="rear_left_wheel"/>
-    <parent link="body_link"/>
+    <parent link="base_link"/>
     <axis xyz="0 1 0" rpy="0 0 0"/>
     <limit effort="1" velocity="10"/>
@@ -255,5 +248,5 @@
     <origin xyz="${scale_bot*-0.055} ${scale_bot*-0.11} 0" rpy="0 0 0"/>
     <child link="rear_right_wheel"/>
-    <parent link="body_link"/>
+    <parent link="base_link"/>
     <axis xyz="0 1 0" rpy="0 0 0"/>
     <limit effort="1" velocity="10"/>
@@ -313,5 +306,5 @@
     <axis xyz="0 1 0" />
     <origin xyz="${scale_bot*0.1} 0 ${scale_bot*0.0584}" rpy="0 0 3.14"/>
-    <parent link="body_link"/>
+    <parent link="base_link"/>
     <child link="laser"/>
   </joint>
@@ -340,5 +333,5 @@
     <axis xyz="0 1 0" />
     <origin xyz="${scale_bot*0.1} ${scale_bot*0.05} ${scale_bot*0.05}" rpy="0 0 0.13 "/>
-    <parent link="body_link"/>
+    <parent link="base_link"/>
     <child link="range_fl"/>
   </joint>
@@ -347,5 +340,5 @@
     <axis xyz="0 1 0" />
     <origin xyz="${scale_bot*0.1} ${scale_bot*-0.05} ${scale_bot*0.01}" rpy="0 0 -0.13 "/>
-    <parent link="body_link"/>
+    <parent link="base_link"/>
     <child link="range_fr"/>
   </joint>
@@ -354,5 +347,5 @@
     <axis xyz="0 1 0" />
     <origin xyz="${scale_bot*-0.1} ${scale_bot*0.05} ${scale_bot*0.01}" rpy="0 0 3.01 "/>
-    <parent link="body_link"/>
+    <parent link="base_link"/>
     <child link="range_rl"/>
   </joint>
@@ -361,5 +354,5 @@
     <axis xyz="0 1 0" />
     <origin xyz="${scale_bot*-0.1} ${scale_bot*-0.05} ${scale_bot*0.01}" rpy="0 0 3.27 "/>
-    <parent link="body_link"/>
+    <parent link="base_link"/>
     <child link="range_rr"/>
   </joint>

File: urdf/youbot_arm/arm.urdf.xacro (robot description, xacro)
@@ -7,5 +7,5 @@
   <xacro:include filename="$(find EXPROBLAB_Assignment2)/urdf/youbot_arm/arm.transmission.xacro" />
   <xacro:include filename="$(find EXPROBLAB_Assignment2)/urdf/youbot_arm/limits.urdf.xacro" />
-  <xacro:property name="scale_robot" value="3.0"/>
+  <xacro:property name="scale_robot" value="1.0"/>
   <xacro:property name="scale" value="${scale_robot*0.5}"/>
   <!-- specifies the offset to include the 10mm table flange and the 3.225cm model offset -->

File: urdf/youbot_arm/limits.urdf.xacro (robot description, xacro)
@@ -3,5 +3,5 @@
   <!-- common properties -->
   <xacro:property name="M_PI" value="3.1415926535897931" />
-  <xacro:property name="scale_robot" value="3.0"/>
+  <xacro:property name="scale_robot" value="1.0"/>
   <xacro:property name="scale" value="${scale_robot*0.5}"/>
   <xacro:property name="threshold" value="${0}" />

Commit message: modification for the laser

File: urdf/rosbot.xacro (robot description, xacro)
@@ -305,5 +305,5 @@
   <joint name="rplidar_joint" type="fixed">
     <axis xyz="0 1 0" />
-    <origin xyz="${scale_bot*0.1} 0 ${scale_bot*0.0584}" rpy="0 0 3.14"/>
+    <origin xyz="${scale_bot*0.1} 0 ${scale_bot*0.0584}" rpy="0 0 0"/>
     <parent link="base_link"/>
     <child link="laser"/>

File: urdf/youbot_arm/arm.urdf.xacro (robot description, xacro)
@@ -42,5 +42,5 @@
     <!-- joint between arm_0_link and arm_1_link -->
     <joint name="${name}_joint_1" type="revolute">
-      <origin xyz="${scale*0.024} 0 ${scale*0.096}" rpy="0 0 0"/>
+      <origin xyz="${scale*0.024} 0 ${scale*0.096}" rpy="0 0 3.14"/>
       <parent link="${name}_link_0"/>
       <child link="${name}_link_1"/>

Commit message: changed color of base_link

File: urdf/rosbot.xacro (robot description, xacro)
@@ -29,4 +29,5 @@
         <mesh filename="package://EXPROBLAB_Assignment2/meshes/box.stl" scale="${scale_bot*0.001} ${scale_bot*0.001} ${scale_bot*0.001}" />
       </geometry>
+      <material name="White"/>
     </visual>
   </link>
@@ -322,5 +323,5 @@
         <mesh filename="package://EXPROBLAB_Assignment2/meshes/rplidar.stl" scale="${scale_bot*0.001} ${scale_bot*0.001} ${scale_bot*0.001}" />
       </geometry>
-      <material name="Black"/>
+      <material name="White"/>
     </visual>
     <inertial>
